File: SlaveDesignFiles/26c32.kicad_sch (KiCad schematic)
At the start: 35 parts

Commit message: 1. 在USB处，修改了type-c5V输入的定义，添加了二极管；2. 将CJA1117B-3.3替换为AMS1117-3.3；3. 分配了testpoint的封装；4. 修改了H485，can插件的PE_GNG引脚定义。
Parts:
- gave numbers to parts that had none: 35

Commit message: Fix bugs in PWM subsheet
Parts:
- renumbered Q28 to D10, Q29 to D11, Q27 to D9, Q30 to Q19
Connections:
- net D+5V_ renamed D+5V
Changed lines of the file:
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@@
 			)
 		)
-		(property "Value" "D+5V_"
+		(property "Value" "D+5V"
 			(at 142.24 53.34 0)
 			(effects
@@
 		(on_board yes)
 		(dnp no)
-		(property "Reference" "Q27"
+		(property "Reference" "D9"
 			(at 23.114 82.55 90)
 			(effects
@@
 			(project "sheet1"
 				(path "/54840d93-b842-4275-b1cb-4ec5510cbfff/46ae6068-d92d-4376-a2bb-12fabee21097"
-					(reference "Q27")
+					(reference "D9")
 					(unit 1)
 				)
 				(path "/54840d93-b842-4275-b1cb-4ec5510cbfff/e2a59e57-e0a7-421f-9f4b-bb850d3277d4"
-					(reference "Q31")
+					(reference "D12")
 					(unit 1)
 				)
@@
 		(on_board yes)
 		(dnp no)
-		(property "Reference" "Q29"
+		(property "Reference" "D11"
 			(at 23.114 148.59 90)
 			(effects
@@
 			(project "sheet1"
 				(path "/54840d93-b842-4275-b1cb-4ec5510cbfff/46ae6068-d92d-4376-a2bb-12fabee21097"
-					(reference "Q29")
+					(reference "D11")
 					(unit 1)
 				)
 				(path "/54840d93-b842-4275-b1cb-4ec5510cbfff/e2a59e57-e0a7-421f-9f4b-bb850d3277d4"
-					(reference "Q33")
+					(reference "D14")
 					(unit 1)
 				)
@@
 		(on_board yes)
 		(dnp no)
-		(property "Reference" "Q30"
+		(property "Reference" "Q19"
 			(at 156.21 68.9102 0)
 			(effects
@@
 			(project "sheet1"
 				(path "/54840d93-b842-4275-b1cb-4ec5510cbfff/46ae6068-d92d-4376-a2bb-12fabee21097"
-					(reference "Q30")
+					(reference "Q19")
 					(unit 1)
 				)
 				(path "/54840d93-b842-4275-b1cb-4ec5510cbfff/e2a59e57-e0a7-421f-9f4b-bb850d3277d4"
-					(reference "Q34")
+					(reference "Q20")
 					(unit 1)
 				)
@@
 		(on_board yes)
 		(dnp no)
-		(property "Reference" "Q28"
+		(property "Reference" "D10"
 			(at 18.542 120.142 90)
 			(effects
@@
 			(project "sheet1"
 				(path "/54840d93-b842-4275-b1cb-4ec5510cbfff/46ae6068-d92d-4376-a2bb-12fabee21097"
-					(reference "Q28")
+					(reference "D10")
 					(unit 1)
 				)
 				(path "/54840d93-b842-4275-b1cb-4ec5510cbfff/e2a59e57-e0a7-421f-9f4b-bb850d3277d4"
-					(reference "Q32")
+					(reference "D13")
 					(unit 1)
 				)
