File: SlaveDesignFiles/IPM.kicad_sch (KiCad schematic)
At the start: 19 parts

Commit message: 1. 在USB处，修改了type-c5V输入的定义，添加了二极管；2. 将CJA1117B-3.3替换为AMS1117-3.3；3. 分配了testpoint的封装；4. 修改了H485，can插件的PE_GNG引脚定义。
Parts:
- gave numbers to parts that had none: 19

Commit message: Fix bugs in PWM subsheet
Parts:
- removed D2: B5819WS, Lib_sheet_10:SOD-323_L1.7-W1.3-LS2.5-FD, symbol sheet1-altium-import:B5819WS_C7420331
- removed R192, R194: 20K/1%, Resistor_SMD:R_0603_1608Metric, symbol sheet1-altium-import:RES_8
- added C107: 15pF/50V, Capacitor_SMD:C_0603_1608Metric, symbol sheet1-altium-import:CAP
- added C108: 0.01uF/50V, Capacitor_SMD:C_0603_1608Metric, symbol sheet1-altium-import:CAP_1
- added D18: LEDRED, LED_SMD:LED_0805_2012Metric, symbol sheet1-altium-import:root_3_LED0
- added Q25: SN74LVC1G125DCKR, Lib2ic:SOT-353_L2.2-W1.4-P0.65-LS2.4-BR, symbol sheet1-altium-import:SN74LVC1G125DCKR
- added Q27: FMMT618TA, Package_TO_SOT_SMD:SOT-23, symbol sheet1-altium-import:root_0_NPN
- added R187: 3.3K, Lib_sheet_10:R_0603_1608Metric, symbol sheet1-altium-import:RES_2
- added R188: 470R, Resistor_SMD:R_0603_1608Metric, symbol sheet1-altium-import:RES_6
- added R195: 62R/1%, Resistor_SMD:R_0603_1608Metric, symbol sheet1-altium-import:RES_4
- added R202: 10K, Resistor_SMD:R_0805_2012Metric, symbol sheet1-altium-import:root_2_Res2
- added R203: 2K, Resistor_SMD:R_0805_2012Metric, symbol sheet1-altium-import:root_3_Res2
- added R204: 1K, Resistor_SMD:R_0805_2012Metric, symbol sheet1-altium-import:root_1_Res2
- renumbered C107 to C109, D1 to D17, Q43 to Q26, R187 to R189, R188 to R190, R189 to R191, R190 to R192, R191 to R193, R193 to R194, R195 to R196, R196 to R197, R197 to R198, R198 to R199, R199 to R200, R200 to R201
Connections:
- net AGND: now also C107.1, C108.1, Q25.1 (OE#), Q25.3 (GND), Q27.2 (E), R203.2; no longer CN3.17
- net DSP_PWM_~{FAULT}: now also CN3.17, R187.2, R188.1, R195.1, R202.2
- net VDD: now also C108.2, Q25.5 (VCC)
- net at Q26.1 (1OE#): now also D17.2 (K), Q26.19 (2OE#)
- net D+5V_ renamed D+5V
- net D+5V: now also D18.1 (A), R187.1
- net IPM_Temperature renamed DSP_Temperature
- net IPM_VDC_BUS renamed DSP_VDC_BUS
- new net: C107.2, Q25.2 (A), R188.2
- new net: Q27.1 (B), R202.1, R203.1
- new net: Q25.4 (Y), R195.2
- new net: D18.2 (K), R204.2
- new net: Q27.3 (C), R204.1
Other:
- note added: "low active for fault and the light will be off"
