File: SlaveDesignFiles/sheet1.kicad_sch (KiCad schematic)
At the start: 143 parts, among them U1 AMS1117-3.3

Commit message: 1. 在USB处，修改了type-c5V输入的定义，添加了二极管；2. 将CJA1117B-3.3替换为AMS1117-3.3；3. 分配了testpoint的封装；4. 修改了H485，can插件的PE_GNG引脚定义。
Parts:
- removed Q?: CJA1117B-3.3, Lib_sheet_10:SOT-89-3_L4.5-W2.5-P1.50-LS4.2-BR, symbol sheet1-altium-import:CJA1117B-3.3
- added D23: SK36A-LTP, Lib_sheet_10:SMA_L4.3-W2.6-LS5.2-RD, symbol sheet1-altium-import:SK36A-LTP
- TP1, TP2: footprint (none) -> TestPoint:TestPoint_Loop_D2.60mm_Drill1.4mm_Beaded
- gave numbers to parts that had none: 139
- renumbered U1 to U8
Connections:
- net +3.3V: now also U8.2 (VO)
- net D+5V: now also Q57.A4B9 (VBUS), Q57.B4A9 (VBUS), D23.2 (A)
- net D+5V_: now also U8.3 (VI), D23.1 (K); no longer Q57.A4B9 (VBUS), Q57.B4A9 (VBUS)
- net PE_GND: no longer CN7.5, CN8.5
- net VDD: no longer U8.2 (VO)
- no-connect marks 91 -> 93
Other:
- moved on the sheet: U8

Commit message: Fix bugs in PWM subsheet
Parts:
- renumbered C111 to C119, C112 to C120, C113 to C121, C114 to C122, C115 to C123, C116 to C124, C117 to C125, C118 to C126, C119 to C127, C120 to C128, C121 to C129, C122 to C130, C123 to C131, C124 to C132, C125 to C133, C126 to C134, C127 to C135, C128 to C136, C129 to C137, C130 to C138, C131 to C139, C132 to C140, C133 to C141, C134 to C142, C135 to C143, C136 to C144, C137 to C145, D9 to D25, D10 to D26, D11 to D27, D12 to D28, D13 to D29, D14 to D30, D15 to D31, Q54 to D32, Q55 to D33, D16 to D34, D17 to D35, D18 to D36, D23 to D37, D19 to D38, D20 to D39, D21 to D40, D22 to D41, L15 to L17, L16 to L18, L17 to L19, Q47 to Q37, Q48 to Q38, Q49 to Q39, Q50 to Q40, Q51 to Q41, Q52 to Q42, Q53 to Q43, Q56 to Q44, U8 to Q45, Q57 to Q46, Q58 to Q47, Q59 to Q48, R243 to R259, R244 to R260, R245 to R261, R246 to R262, R247 to R263, R248 to R264, R249 to R265, R250 to R266, R251 to R267, R252 to R268, R253 to R269, R254 to R270, R255 to R271, R256 to R272, R257 to R273, R258 to R274, R259 to R275, R260 to R276, R261 to R277, R262 to R278, R263 to R279, R264 to R280, R265 to R281, R266 to R282, R267 to R283, R268 to R284, R269 to R285, R270 to R286, R271 to R287, R272 to R288, R273 to R289, R274 to R290, R275 to R291, R276 to R292, R277 to R293, R278 to R294, R279 to R295, R280 to R296, R281 to R297, R282 to R298, R283 to R299, R284 to R300, R285 to R301, R286 to R302, R287 to R303, R288 to R304, R289 to R305, R290 to R306, R291 to R307, R292 to R308
Connections:
- net +3.3V is gone; now on net VDD: C142.1, C143.2, C144.1, J5.1, J5.2, J6.1, J6.2, Q45.2 (VO)
- net D+5V_ is gone; now on net D+5V: C126.1, C127.1, C138.2, C140.1, D25.1 (A), D26.1 (A), D27.1 (A), D30.1 (A), D31.1 (K), D37.1 (K), DSUB1.1, DSUB2.1, DSUB3.1, DSUB4.1, DSUB5.1, J7.11, J7.12, J7.13, J7.14, Q42.3 (VCC), Q43.3 (VCC), Q44.7 (VREGIN), Q44.8 (VBUS), Q45.3 (VI), Q48.5 (VCC), R291.2, R293.2, R295.2, U1.1 (5V), U2.11 (5V), U2.12 (5V), U2.13 (5V), U2.14 (5V), U2.15 (5V), U2.16 (5V), U3.1 (5V), U3.29 (5V), U3.30 (5V), U3.31 (5V), U3.32 (5V), U4.40 (5V), U5.1 (5V), U5.40 (5V), U6.1 (5V)
- net D+5V: no longer D31.2 (A), D37.2 (A), J3.10, J3.7, J3.8, J3.9, Q46.A4B9 (VBUS), Q46.B4A9 (VBUS)
- net VDD: no longer U3.25 (3.3V), U3.26 (3.3V), U3.27 (3.3V), U3.28 (3.3V)
- net ADC_CLK_1 renamed ADC_CLK_X1
- net ADC_CLK_2 renamed ADC_CLK_X2
- net IPM_Temperature1 renamed DSP_Temperature1
- net IPM_Temperature2 renamed DSP_Temperature2
- net IPM_Temperature3 renamed DSP_Temperature3
- net IPM_Temperature4 renamed DSP_Temperature4
- net IPM_VDC_BUS1 renamed DSP_VDC_BUS1
- net IPM_VDC_BUS2 renamed DSP_VDC_BUS2
- net IPM_VDC_BUS3 renamed DSP_VDC_BUS3
- net IPM_VDC_BUS4 renamed DSP_VDC_BUS4
- new net Header-D+5V: D31.2 (A), J3.10, J3.7, J3.8, J3.9
- new net USB_D+5V: D37.2 (A), Q46.A4B9 (VBUS), Q46.B4A9 (VBUS)
- no-connect marks 93 -> 97
Other:
- sheet IPM1 ports: added DSP_Temperature, DSP_VDC_BUS; removed IPM_Temperature, IPM_VDC_BUS
- sheet IPM2 ports: added DSP_Temperature, DSP_VDC_BUS; removed IPM_Temperature, IPM_VDC_BUS
- sheet IPM3 ports: added DSP_Temperature, DSP_VDC_BUS; removed IPM_Temperature, IPM_VDC_BUS
- sheet IPM4 ports: added DSP_Temperature, DSP_VDC_BUS; removed IPM_Temperature, IPM_VDC_BUS
- note added: "电流采样用的20MHz时钟"
- note added: "绝对值编码器CLB实现多摩川协议tformat）（本质上是用SPI外外设实现的！"
- note removed: "绝对值编码器CLB实现多摩川协议tformat"
